Commit message: [wip]changed to allow only some nodes to be full order dynamics. fixed bug when there were multiple contacts on the same joint.

File: tests/test_data/achilles.urdf (robot description, URDF)
Before this commit: robot achilles, 29 links, 28 joints
Links:
- added link foot_front_left
- added link foot_front_right
- added link foot_rear_left
- added link foot_rear_right
Joints:
- added joint foot_front_left_joint: type fixed, parent left_ankle_pitch, child foot_front_left, origin xyz=0.088 0 -0.018 rpy=0 0 0
- added joint foot_front_right_joint: type fixed, parent right_ankle_pitch, child foot_front_right, origin xyz=0.088 0 -0.018 rpy=0 0 0
- added joint foot_rear_left_joint: type fixed, parent left_ankle_pitch, child foot_rear_left, origin xyz=-0.02 0 -0.018 rpy=0 0 0
- added joint foot_rear_right_joint: type fixed, parent right_ankle_pitch, child foot_rear_right, origin xyz=-0.02 0 -0.018 rpy=0 0 0

Commit message: added an updated force target

File: tests/test_data/achilles.urdf (robot description, URDF)
Before this commit: robot achilles, 33 links, 32 joints
Joints:
- joint right_hip_pitch_joint: limit lower=-1.5 upper=1.5 effort=35.0 velocity=20 -> lower=-1.5 upper=0.5 effort=35.0 velocity=20

Commit message: added predicition delay comp. started adding raibert

File: tests/test_data/achilles.urdf (robot description, URDF)
Before this commit: robot achilles, 33 links, 32 joints
Joints:
- joint left_ankle_pitch_joint: limit lower=-1 upper=1 effort=35 velocity=20 -> lower=-1 upper=1 effort=35 velocity=2
- joint left_elbow_pitch_joint: limit lower=-1.58 upper=0 effort=24 velocity=10 -> lower=-1.58 upper=0 effort=24 velocity=1
- joint left_hip_pitch_joint: limit lower=-1.5 upper=0.5 effort=35.0 velocity=20 -> lower=-1.5 upper=0.5 effort=35.0 velocity=2
- joint left_hip_roll_joint: limit lower=-1 upper=1 effort=70.0 velocity=10 -> lower=-1 upper=1 effort=70.0 velocity=1
- joint left_hip_yaw_joint: limit lower=-1 upper=1 effort=35.0 velocity=20 -> lower=-1 upper=1 effort=35.0 velocity=2
- joint left_knee_pitch_joint: limit lower=0 upper=2 effort=70.0 velocity=10 -> lower=0 upper=2 effort=70.0 velocity=1
- joint left_shoulder_pitch_joint: limit lower=-1.58 upper=1.58 effort=35 velocity=20 -> lower=-1.58 upper=1.58 effort=35 velocity=2
- joint left_shoulder_roll_joint: limit lower=0 upper=3.141592653589793 effort=12 velocity=20 -> lower=0 upper=3.141592653589793 effort=12 velocity=2
- joint left_shoulder_yaw_joint: limit lower=-1.58 upper=1.58 effort=12 velocity=20 -> lower=-1.58 upper=1.58 effort=12 velocity=2
- joint right_ankle_pitch_joint: limit lower=-1 upper=1 effort=35 velocity=20 -> lower=-1 upper=1 effort=35 velocity=2
- joint right_elbow_pitch_joint: limit lower=-1.58 upper=0 effort=24 velocity=20 -> lower=-1.58 upper=0 effort=24 velocity=2
- joint right_hip_pitch_joint: limit lower=-1.5 upper=0.5 effort=35.0 velocity=20 -> lower=-1.5 upper=0.5 effort=35.0 velocity=2
- joint right_hip_roll_joint: limit lower=-1 upper=1 effort=70.0 velocity=10 -> lower=-1 upper=1 effort=70.0 velocity=1
- joint right_hip_yaw_joint: limit lower=-1 upper=1 effort=35.0 velocity=20 -> lower=-1 upper=1 effort=35.0 velocity=2
- joint right_knee_pitch_joint: limit lower=0 upper=2 effort=70.0 velocity=10 -> lower=0 upper=2 effort=70.0 velocity=1
- joint right_shoulder_pitch_joint: limit lower=-1.58 upper=1.58 effort=35 velocity=20 -> lower=-1.58 upper=1.58 effort=35 velocity=2
- joint right_shoulder_roll_joint: limit lower=-3.14 upper=0 effort=35 velocity=20 -> lower=-3.14 upper=0 effort=35 velocity=2
- joint right_shoulder_yaw_joint: limit lower=-1.58 upper=1.58 effort=12.0 velocity=20 -> lower=-1.58 upper=1.58 effort=12.0 velocity=2
