Commit message: corresponding commit for biped basic walking in sim

File: tests/test_data/g1_hand_v2.urdf (robot description, URDF)
Before this commit: robot g1_29dof_with_hand, 57 links, 56 joints
Links:
- added link ll_heel
- added link ll_toe
- added link lr_heel
- added link lr_toe
- added link rl_heel
- added link rl_toe
- added link rr_heel
- added link rr_toe
- link head_link: geometry collision mesh filename=package://g1_model/meshes/head_link.STL; visual mesh filename=package://g1_model/meshes/head_link.STL
- link left_ankle_pitch_link: geometry collision mesh filename=package://g1_model/meshes/left_ankle_pitch_link.STL; visual mesh filename=package://g1_model/meshes/left_ankle_pitch_link.STL
- link left_ankle_roll_link: geometry collision sphere radius=0.005; collision sphere radius=0.005
- link left_elbow_link: geometry collision mesh filename=package://g1_model/meshes/left_elbow_link.STL; visual mesh filename=package://g1_model/meshes/left_elbow_link.STL
- link left_hand_index_0_link: geometry collision mesh filename=package://g1_model/meshes/left_hand_index_0_link.STL; visual mesh filename=package://g1_model/meshes/left_hand_index_0_link.STL
- link left_hand_index_1_link: geometry collision mesh filename=package://g1_model/meshes/left_hand_index_1_link.STL; visual mesh filename=package://g1_model/meshes/left_hand_index_1_link.STL
- link left_hand_middle_0_link: geometry collision mesh filename=package://g1_model/meshes/left_hand_middle_0_link.STL; visual mesh filename=package://g1_model/meshes/left_hand_middle_0_link.STL
- link left_hand_middle_1_link: geometry collision mesh filename=package://g1_model/meshes/left_hand_middle_1_link.STL; visual mesh filename=package://g1_model/meshes/left_hand_middle_1_link.STL
- link left_hand_palm_link: geometry collision mesh filename=package://g1_model/meshes/left_hand_palm_link.STL; visual mesh filename=package://g1_model/meshes/left_hand_palm_link.STL
- link left_hand_thumb_0_link: geometry collision mesh filename=package://g1_model/meshes/left_hand_thumb_0_link.STL; visual mesh filename=package://g1_model/meshes/left_hand_thumb_0_link.STL
- link left_hand_thumb_1_link: geometry collision box size=0.02 0.03 0.02; visual mesh filename=package://g1_model/meshes/left_hand_thumb_1_link.STL
- link left_hand_thumb_2_link: geometry collision mesh filename=package://g1_model/meshes/left_hand_thumb_2_link.STL; visual mesh filename=package://g1_model/meshes/left_hand_thumb_2_link.STL
- link left_hip_pitch_link: geometry collision mesh filename=package://g1_model/meshes/left_hip_pitch_link.STL; visual mesh filename=package://g1_model/meshes/left_hip_pitch_link.STL
- link left_hip_roll_link: geometry collision mesh filename=package://g1_model/meshes/left_hip_roll_link.STL; visual mesh filename=package://g1_model/meshes/left_hip_roll_link.STL
- link left_hip_yaw_link: geometry collision mesh filename=package://g1_model/meshes/left_hip_yaw_link.STL; visual mesh filename=package://g1_model/meshes/left_hip_yaw_link.STL
- link left_knee_link: geometry collision mesh filename=package://g1_model/meshes/left_knee_link.STL; visual mesh filename=package://g1_model/meshes/left_knee_link.STL
- link left_shoulder_pitch_link: geometry collision cylinder length=0.05 radius=0.03; visual mesh filename=package://g1_model/meshes/left_shoulder_pitch_link.STL
- link left_shoulder_roll_link: geometry collision cylinder length=0.03 radius=0.03; visual mesh filename=package://g1_model/meshes/left_shoulder_roll_link.STL
- link left_shoulder_yaw_link: geometry collision mesh filename=package://g1_model/meshes/left_shoulder_yaw_link.STL; visual mesh filename=package://g1_model/meshes/left_shoulder_yaw_link.STL
- link left_wrist_pitch_link: geometry collision mesh filename=package://g1_model/meshes/left_wrist_pitch_link.STL; visual mesh filename=package://g1_model/meshes/left_wrist_pitch_link.STL
- link left_wrist_roll_link: geometry collision mesh filename=package://g1_model/meshes/left_wrist_roll_link.STL; visual mesh filename=package://g1_model/meshes/left_wrist_roll_link.STL
- link left_wrist_yaw_link: geometry collision mesh filename=package://g1_model/meshes/left_wrist_yaw_link.STL; visual mesh filename=package://g1_model/meshes/left_wrist_yaw_link.STL
- link logo_link: geometry collision mesh filename=package://g1_model/meshes/logo_link.STL; visual mesh filename=package://g1_model/meshes/logo_link.STL
- link pelvis: geometry visual mesh filename=package://g1_model/meshes/pelvis.STL
- link pelvis_contour_link: geometry collision mesh filename=package://g1_model/meshes/pelvis_contour_link.STL; visual mesh filename=package://g1_model/meshes/pelvis_contour_link.STL
- link right_ankle_pitch_link: geometry collision mesh filename=package://g1_model/meshes/right_ankle_pitch_link.STL; visual mesh filename=package://g1_model/meshes/right_ankle_pitch_link.STL
- link right_ankle_roll_link: geometry collision sphere radius=0.005; collision sphere radius=0.005
- link right_elbow_link: geometry collision mesh filename=package://g1_model/meshes/right_elbow_link.STL; visual mesh filename=package://g1_model/meshes/right_elbow_link.STL
- link right_hand_index_0_link: geometry collision mesh filename=package://g1_model/meshes/right_hand_index_0_link.STL; visual mesh filename=package://g1_model/meshes/right_hand_index_0_link.STL
- link right_hand_index_1_link: geometry collision mesh filename=package://g1_model/meshes/right_hand_index_1_link.STL; visual mesh filename=package://g1_model/meshes/right_hand_index_1_link.STL
- link right_hand_middle_0_link: geometry collision mesh filename=package://g1_model/meshes/right_hand_middle_0_link.STL; visual mesh filename=package://g1_model/meshes/right_hand_middle_0_link.STL
- link right_hand_middle_1_link: geometry collision mesh filename=package://g1_model/meshes/right_hand_middle_1_link.STL; visual mesh filename=package://g1_model/meshes/right_hand_middle_1_link.STL
- link right_hand_palm_link: geometry collision mesh filename=package://g1_model/meshes/right_hand_palm_link.STL; visual mesh filename=package://g1_model/meshes/right_hand_palm_link.STL
- link right_hand_thumb_0_link: geometry collision mesh filename=package://g1_model/meshes/right_hand_thumb_0_link.STL; visual mesh filename=package://g1_model/meshes/right_hand_thumb_0_link.STL
- link right_hand_thumb_1_link: geometry collision box size=0.02 0.03 0.02; visual mesh filename=package://g1_model/meshes/right_hand_thumb_1_link.STL
- link right_hand_thumb_2_link: geometry collision mesh filename=package://g1_model/meshes/right_hand_thumb_2_link.STL; visual mesh filename=package://g1_model/meshes/right_hand_thumb_2_link.STL
- link right_hip_pitch_link: geometry collision mesh filename=package://g1_model/meshes/right_hip_pitch_link.STL; visual mesh filename=package://g1_model/meshes/right_hip_pitch_link.STL
- link right_hip_roll_link: geometry collision mesh filename=package://g1_model/meshes/right_hip_roll_link.STL; visual mesh filename=package://g1_model/meshes/right_hip_roll_link.STL
- link right_hip_yaw_link: geometry collision mesh filename=package://g1_model/meshes/right_hip_yaw_link.STL; visual mesh filename=package://g1_model/meshes/right_hip_yaw_link.STL
- link right_knee_link: geometry collision mesh filename=package://g1_model/meshes/right_knee_link.STL; visual mesh filename=package://g1_model/meshes/right_knee_link.STL
- link right_shoulder_pitch_link: geometry collision cylinder length=0.05 radius=0.03; visual mesh filename=package://g1_model/meshes/right_shoulder_pitch_link.STL
- link right_shoulder_roll_link: geometry collision cylinder length=0.03 radius=0.03; visual mesh filename=package://g1_model/meshes/right_shoulder_roll_link.STL
- link right_shoulder_yaw_link: geometry collision mesh filename=package://g1_model/meshes/right_shoulder_yaw_link.STL; visual mesh filename=package://g1_model/meshes/right_shoulder_yaw_link.STL
- link right_wrist_pitch_link: geometry collision mesh filename=package://g1_model/meshes/right_wrist_pitch_link.STL; visual mesh filename=package://g1_model/meshes/right_wrist_pitch_link.STL
- link right_wrist_roll_link: geometry collision mesh filename=package://g1_model/meshes/right_wrist_roll_link.STL; visual mesh filename=package://g1_model/meshes/right_wrist_roll_link.STL
- link right_wrist_yaw_link: geometry collision mesh filename=package://g1_model/meshes/right_wrist_yaw_link.STL; visual mesh filename=package://g1_model/meshes/right_wrist_yaw_link.STL
- link torso_link: geometry collision mesh filename=package://g1_model/meshes/torso_link.STL; visual mesh filename=package://g1_model/meshes/torso_link.STL
- link waist_roll_link: geometry visual mesh filename=package://g1_model/meshes/waist_roll_link.STL
- link waist_support_link: geometry collision mesh filename=package://g1_model/meshes/waist_support_link.STL; visual mesh filename=package://g1_model/meshes/waist_support_link.STL
- link waist_yaw_link: geometry visual mesh filename=package://g1_model/meshes/waist_yaw_link.STL
Joints:
- added joint ll_heel_joint: type fixed, parent left_ankle_roll_link, child ll_heel, origin xyz=-0.05 0.025 -0.03 rpy=0 0 0
- added joint ll_toe_joint: type fixed, parent left_ankle_roll_link, child ll_toe, origin xyz=0.12 0.03 -0.03 rpy=0 0 0
- added joint lr_heel_joint: type fixed, parent left_ankle_roll_link, child lr_heel, origin xyz=-0.05 -0.025 -0.03 rpy=0 0 0
- added joint lr_toe_joint: type fixed, parent left_ankle_roll_link, child lr_toe, origin xyz=0.12 -0.03 -0.03 rpy=0 0 0
- added joint rl_heel_joint: type fixed, parent left_ankle_roll_link, child rl_heel, origin xyz=-0.05 0.025 -0.03 rpy=0 0 0
- added joint rl_toe_joint: type fixed, parent left_ankle_roll_link, child rl_toe, origin xyz=0.12 0.03 -0.03 rpy=0 0 0
- added joint rr_heel_joint: type fixed, parent left_ankle_roll_link, child rr_heel, origin xyz=-0.05 -0.025 -0.03 rpy=0 0 0
- added joint rr_toe_joint: type fixed, parent left_ankle_roll_link, child rr_toe, origin xyz=0.12 -0.03 -0.03 rpy=0 0 0
- joint left_ankle_pitch_joint: limit lower=-0.87267 upper=0.5236 effort=50 velocity=37 -> lower=-0.87267 upper=0.5236 effort=50 velocity=12
- joint left_ankle_roll_joint: limit lower=-0.2618 upper=0.2618 effort=50 velocity=37 -> lower=-0.2618 upper=0.2618 effort=50 velocity=12
- joint left_elbow_joint: limit lower=-1.0472 upper=2.0944 effort=25 velocity=37 -> lower=-1.0472 upper=2.0944 effort=25 velocity=12
- joint left_hip_pitch_joint: limit lower=-2.5307 upper=2.8798 effort=88 velocity=32 -> lower=-2.5307 upper=2.8798 effort=88 velocity=12
- joint left_hip_roll_joint: limit lower=-0.5236 upper=2.9671 effort=88 velocity=32 -> lower=-0.5236 upper=2.9671 effort=88 velocity=12
- joint left_hip_yaw_joint: limit lower=-2.7576 upper=2.7576 effort=88 velocity=32 -> lower=-2.7576 upper=2.7576 effort=88 velocity=12
- joint left_knee_joint: limit lower=-0.087267 upper=2.8798 effort=139 velocity=20 -> lower=-0.087267 upper=2.8798 effort=139 velocity=12
- joint left_shoulder_pitch_joint: limit lower=-3.0892 upper=2.6704 effort=25 velocity=37 -> lower=-3.0892 upper=2.6704 effort=25 velocity=12
- joint left_shoulder_roll_joint: limit lower=-1.5882 upper=2.2515 effort=25 velocity=37 -> lower=-1.5882 upper=2.2515 effort=25 velocity=12
- joint left_shoulder_yaw_joint: limit lower=-2.618 upper=2.618 effort=25 velocity=37 -> lower=-2.618 upper=2.618 effort=25 velocity=12
- joint left_wrist_roll_joint: limit lower=-1.972222054 upper=1.972222054 effort=25 velocity=37 -> lower=-1.972222054 upper=1.972222054 effort=25 velocity=12
- joint right_ankle_pitch_joint: limit lower=-0.87267 upper=0.5236 effort=50 velocity=37 -> lower=-0.87267 upper=0.5236 effort=50 velocity=12
- joint right_ankle_roll_joint: limit lower=-0.2618 upper=0.2618 effort=50 velocity=37 -> lower=-0.2618 upper=0.2618 effort=50 velocity=12
- joint right_elbow_joint: limit lower=-1.0472 upper=2.0944 effort=25 velocity=37 -> lower=-1.0472 upper=2.0944 effort=25 velocity=12
- joint right_hip_pitch_joint: limit lower=-2.5307 upper=2.8798 effort=88 velocity=32 -> lower=-2.5307 upper=2.8798 effort=88 velocity=12
- joint right_hip_roll_joint: limit lower=-2.9671 upper=0.5236 effort=88 velocity=32 -> lower=-2.9671 upper=0.5236 effort=88 velocity=12
- joint right_hip_yaw_joint: limit lower=-2.7576 upper=2.7576 effort=88 velocity=32 -> lower=-2.7576 upper=2.7576 effort=88 velocity=12
- joint right_knee_joint: limit lower=-0.087267 upper=2.8798 effort=139 velocity=20 -> lower=-0.087267 upper=2.8798 effort=139 velocity=12
- joint right_shoulder_pitch_joint: limit lower=-3.0892 upper=2.6704 effort=25 velocity=37 -> lower=-3.0892 upper=2.6704 effort=25 velocity=12
- joint right_shoulder_roll_joint: limit lower=-2.2515 upper=1.5882 effort=25 velocity=37 -> lower=-2.2515 upper=1.5882 effort=25 velocity=12
- joint right_shoulder_yaw_joint: limit lower=-2.618 upper=2.618 effort=25 velocity=37 -> lower=-2.618 upper=2.618 effort=25 velocity=12
- joint right_wrist_roll_joint: limit lower=-1.972222054 upper=1.972222054 effort=25 velocity=37 -> lower=-1.972222054 upper=1.972222054 effort=25 velocity=12
- joint waist_pitch_joint: limit lower=-0.52 upper=0.52 effort=50 velocity=37 -> lower=-0.52 upper=0.52 effort=50 velocity=12
- joint waist_roll_joint: limit lower=-0.52 upper=0.52 effort=50 velocity=37 -> lower=-0.52 upper=0.52 effort=50 velocity=12
- joint waist_yaw_joint: limit lower=-2.618 upper=2.618 effort=88 velocity=32 -> lower=-2.618 upper=2.618 effort=88 velocity=12

Commit message: corresponding commit for the humanoid doing stepping stones in sim. added polytope specific frames to optimize with

File: tests/test_data/g1_hand_v2.urdf (robot description, URDF)
Before this commit: robot g1_29dof_with_hand, 65 links, 64 joints
Links:
- added link left_foot_middle
- added link right_foot_middle
Joints:
- added joint left_foot_middle_joint: type fixed, parent left_ankle_roll_link, child left_foot_middle, origin xyz=0.035 0 -0.03 rpy=0 0 0
- added joint right_foot_middle_joint: type fixed, parent right_ankle_roll_link, child right_foot_middle, origin xyz=0.035 0 -0.03 rpy=0 0 0
